File: tinyPEPPER.kicad_pcb (KiCad board)
At the start: 2 copper layers, 20 x 20 mm, 97 parts, among them U201 EFM8BB10, U301 EFM8BB10, U401 EFM8BB10, U501 EFM8BB10

Commit message: cleanup to custom parts
Parts:
- C202, C302, C402, C502: footprint Resistors_SMD:R_0402 -> custom:C_0402_CUSTOM
- R201, R202, R203, R204, R205, R206, R207, R301, R302, R303, R304, R305, R306, R307, R401, R402, R403, R404, R405, R406, R407, R501, R502, R503, R504, R505, R506, R507: footprint Resistors_SMD:R_0402 -> custom:R_0402_CUSTOM

Commit message: phase tabs
Parts:
- removed the G*** at (114.2, 103.7)
- G***: moved to B.Cu
- moved OUT_A501 2.31 mm to (102.9, 120.4)
- moved OUT_A401 2.31 mm to (102.9, 99.6)
- moved OUT_A301 2.30 mm to (117.1, 120.4)
- moved OUT_A201 2.30 mm to (117.1, 99.6)
- moved OUT_B301 1.67 mm to (114.3, 120.4)
- moved OUT_B501 1.67 mm to (105.7, 120.4)
- moved OUT_B401 1.66 mm to (105.7, 99.6)
- moved OUT_B201 1.65 mm to (114.3, 99.6)
- moved OUT_C301 1.24 mm to (111.5, 120.4)
- moved OUT_C501 1.24 mm to (108.5, 120.4)
- moved OUT_C401 1.22 mm to (108.5, 99.6)
- moved OUT_C201 1.22 mm to (111.5, 99.6)
- moved G*** 0.50 mm to (110.0, 101.3), turned to 0 degrees
Routing:
- net /single esc 4/PHASE_A_0: track 24.8 -> 21.6 mm, vias 3 -> 1
- net /single esc 3/PHASE_B_0: track 12.1 -> 14.9 mm
- net /single esc 1/PHASE_B_0: track 13.8 -> 15.2 mm, vias 2 -> 0
- net /single esc 2/PHASE_B_0: track 10.8 -> 12.1 mm, vias 1 -> 0
- net /single esc 4/PHASE_B_0: track 15.6 -> 14.3 mm, vias 2 -> 0
- net /single esc 1/PHASE_A_0: track 23.5 -> 22.4 mm, vias 3 -> 1
- net /single esc 1/PHASE_C_0: track 11.8 -> 13.0 mm
- net /single esc 3/PHASE_C_0: track 9.30 -> 10.5 mm
- net /single esc 2/PHASE_A_0: track 23.2 -> 24.2 mm
- net /single esc 4/PHASE_C_0: track 13.5 -> 14.2 mm
- net /single esc 3/PHASE_A_0: track 22.3 -> 21.6 mm
Other:
- board size 20 x 20 mm -> 20 x 22.6 mm
- board text added: "03/2017"
- board text added: "REV 0.4"
- board text added: "tinyPEPPER"
- board text removed: "02/2017"
- board text removed: "REV 0.3"
